File: kicad/vfdclock/vfdclock.kicad_pcb (KiCad board)
At the start: 2 copper layers, 72 x 47 mm, 21 parts, among them J1 DC12V, SW1 CLR-SEC, SW2 UP-HOUR, SW3 UP-MIN, SW4 SW_SPDT, SW5 SW_SPDT, U1 T3605, U2 VFD-48C, U3 MC7905, Y2 4.1943MHz

Commit message: Fixed bug
Connections:
- SW4 pad 1: VCC -> unconnected-(SW4-A-Pad1)
Routing:
- net VCC: track 116.8 -> 114.6 mm
Changed lines of the file:
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@@
 	(net 48 "unconnected-(U2-NC-Pad19)")
 	(net 49 "unconnected-(U2-NC-Pad27)")
+	(net 50 "unconnected-(SW4-A-Pad1)")
 	(footprint "Diode_THT:D_A-405_P7.62mm_Horizontal"
 		(layer "F.Cu")
@@
 			(layers "*.Cu" "*.Mask")
 			(remove_unused_layers no)
-			(net 4 "VCC")
+			(net 50 "unconnected-(SW4-A-Pad1)")
 			(pinfunction "A")
-			(pintype "passive")
+			(pintype "passive+no_connect")
 		)
 		(pad "2" thru_hole oval
@@
 	)
 	(segment
-		(start 171.62 111.315)
-		(end 172.7224 110.2126)
+		(start 172.7224 110.2126)
+		(end 171.62 109.1102)
+		(width 0.2)
+		(layer "B.Cu")
+		(net 4)
+	)
+	(segment
+		(start 171.62 109.1102)
+		(end 171.62 105.225)
 		(width 0.2)
 		(layer "B.Cu")
@@
 		(width 0.2)
 		(layer "B.Cu")
-		(net 4)
-	)
-	(segment
-		(start 171.62 105.225)
-		(end 171.62 111.315)
-		(width 0.2)
-		(layer "B.Cu")
