File: kicad/vfdclock/vfdclock.kicad_sch (KiCad schematic)
At the start: 18 parts, among them J1 DC12V, SW1 CLR-SEC, SW2 UP-HOUR, SW3 UP-MIN, SW4 SW_SPDT, SW5 SW_SPDT, U1 T3605, U2 VFD-48C, U3 MC7905, Y2 4.1943MHz

Commit message: Fixed bug
Connections:
- net VCC: no longer SW4.1 (A)
- no-connect marks 1 -> 2
Changed lines of the file:
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@@
-	)
-	(junction
-		(at 54.61 83.82)
-		(diameter 0)
-		(color 0 0 0 0)
 	)
 	(junction
@@
 		(diameter 0)
 		(color 0 0 0 0)
+	)
+	(no_connect
+		(at 58.42 83.82)
 	)
 	(no_connect
@@
 		)
 		(stroke
-			(width 0)
-			(type default)
-		)
-	)
-	(wire
-		(pts
-			(xy 54.61 83.82) (xy 58.42 83.82)
-		)
-		(stroke

Commit message: Updated comments
Other:
- note added: "SW4は表示/非表示の切り替え SW5は２段階の明るさ調節用"
- note removed: "SW4とSW5は連動。２段階の明るさ調節用"
Changed lines of the file:
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@@
 		)
 	)
-	(text "SW4とSW5は連動。２段階の明るさ調節用"
+	(text "SW4は表示/非表示の切り替え\nSW5は２段階の明るさ調節用"
 		(exclude_from_sim no)
 		(at 62.738 111.252 0)
